File: RF_HID_module_test/USB.kicad_sch (KiCad schematic)
At the start: 4 parts, among them J3 CH_USB_C, U3 USBLC6-2SC6

Commit message: Layout V0
Parts:
- FL1: footprint Marijn_KiCad:ACM2012_TDK_UPDATE -> Marijn_KiCad:ACM2012_900_2P_T002_Correct
- J6: renamed from J3; footprint (none) -> Connector_USB:USB_C_Receptacle_HCTL_HC-TYPE-C-16P-01A
- R12: renamed from R3; footprint (none) -> Resistor_SMD:R_0603_1608Metric
- renumbered U3 to U6
Changed lines of the file:
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@@
 		(on_board yes)
 		(dnp no)
-		(property "Reference" "U3"
+		(property "Reference" "U6"
 			(at 94.234 59.436 0)
 			(effects
@@
 			(project "RF_HID_module_test"
 				(path "/32b1f824-104d-4f37-b265-1c31215c2fe4/3052776d-f0df-4f5c-b23a-46f73ae78b94"
-					(reference "U3")
-					(unit 1)
-				)
-				(path "/32b1f824-104d-4f37-b265-1c31215c2fe4/35fb170e-cc4d-4774-8b9f-87fa9e2bb590"
-					(reference "U4")
+					(reference "U6")
+					(unit 1)
+				)
+				(path "/32b1f824-104d-4f37-b265-1c31215c2fe4/35fb170e-cc4d-4774-8b9f-87fa9e2bb590"
+					(reference "U7")
 					(unit 1)
 				)
@@
 		(on_board yes)
 		(dnp no)
-		(property "Reference" "R3"
+		(property "Reference" "R12"
 			(at 82.55 52.832 90)
 			(effects
@@
 			)
 		)
-		(property "Footprint" ""
+		(property "Footprint" "Resistor_SMD:R_0603_1608Metric"
 			(at 82.55 54.61 0)
 			(effects
@@
 			(project ""
 				(path "/32b1f824-104d-4f37-b265-1c31215c2fe4/3052776d-f0df-4f5c-b23a-46f73ae78b94"
-					(reference "R3")
-					(unit 1)
-				)
-				(path "/32b1f824-104d-4f37-b265-1c31215c2fe4/35fb170e-cc4d-4774-8b9f-87fa9e2bb590"
-					(reference "R4")
+					(reference "R12")
+					(unit 1)
+				)
+				(path "/32b1f824-104d-4f37-b265-1c31215c2fe4/35fb170e-cc4d-4774-8b9f-87fa9e2bb590"
+					(reference "R13")
 					(unit 1)
 				)
@@
 		(on_board yes)
 		(dnp no)
-		(property "Reference" "#PWR021"
+		(property "Reference" "#PWR047"
 			(at 93.98 77.47 0)
 			(effects
@@
 			(project "RF_HID_module_test"
 				(path "/32b1f824-104d-4f37-b265-1c31215c2fe4/3052776d-f0df-4f5c-b23a-46f73ae78b94"
-					(reference "#PWR021")
-					(unit 1)
-				)
-				(path "/32b1f824-104d-4f37-b265-1c31215c2fe4/35fb170e-cc4d-4774-8b9f-87fa9e2bb590"
-					(reference "#PWR026")
+					(reference "#PWR047")
+					(unit 1)
+				)
+				(path "/32b1f824-104d-4f37-b265-1c31215c2fe4/35fb170e-cc4d-4774-8b9f-87fa9e2bb590"
+					(reference "#PWR052")
 					(unit 1)
 				)
@@
 		(on_board yes)
 		(dnp no)
-		(property "Reference" "#PWR019"
+		(property "Reference" "#PWR045"
 			(at 91.44 54.61 0)
 			(effects
@@
 			(project "RF_HID_module_test"
 				(path "/32b1f824-104d-4f37-b265-1c31215c2fe4/3052776d-f0df-4f5c-b23a-46f73ae78b94"
-					(reference "#PWR019")
-					(unit 1)
-				)
-				(path "/32b1f824-104d-4f37-b265-1c31215c2fe4/35fb170e-cc4d-4774-8b9f-87fa9e2bb590"
-					(reference "#PWR024")
+					(reference "#PWR045")
+					(unit 1)
+				)
+				(path "/32b1f824-104d-4f37-b265-1c31215c2fe4/35fb170e-cc4d-4774-8b9f-87fa9e2bb590"
+					(reference "#PWR050")
 					(unit 1)
 				)
@@
 		(on_board yes)
 		(dnp no)
-		(property "Reference" "#PWR018"
+		(property "Reference" "#PWR044"
 			(at 78.74 50.8 0)
 			(effects
@@
 			(project "RF_HID_module_test"
 				(path "/32b1f824-104d-4f37-b265-1c31215c2fe4/3052776d-f0df-4f5c-b23a-46f73ae78b94"
-					(reference "#PWR018")
-					(unit 1)
-				)
-				(path "/32b1f824-104d-4f37-b265-1c31215c2fe4/35fb170e-cc4d-4774-8b9f-87fa9e2bb590"
-					(reference "#PWR023")
+					(reference "#PWR044")
+					(unit 1)
+				)
+				(path "/32b1f824-104d-4f37-b265-1c31215c2fe4/35fb170e-cc4d-4774-8b9f-87fa9e2bb590"
+					(reference "#PWR049")
 					(unit 1)
 				)
@@
 		(on_board yes)
 		(dnp no)
-		(property "Reference" "#PWR022"
+		(property "Reference" "#PWR048"
 			(at 62.23 92.71 0)
 			(effects
@@
 			(project "RF_HID_module_test"
 				(path "/32b1f824-104d-4f37-b265-1c31215c2fe4/3052776d-f0df-4f5c-b23a-46f73ae78b94"
-					(reference "#PWR022")
-					(unit 1)
-				)
-				(path "/32b1f824-104d-4f37-b265-1c31215c2fe4/35fb170e-cc4d-4774-8b9f-87fa9e2bb590"
-					(reference "#PWR027")
+					(reference "#PWR048")
+					(unit 1)
+				)
+				(path "/32b1f824-104d-4f37-b265-1c31215c2fe4/35fb170e-cc4d-4774-8b9f-87fa9e2bb590"
+					(reference "#PWR053")
 					(unit 1)
 				)
@@
 		(on_board yes)
 		(dnp no)
-		(property "Reference" "#PWR020"
+		(property "Reference" "#PWR046"
 			(at 93.98 62.23 0)
 			(effects
@@
 			(project "RF_HID_module_test"
 				(path "/32b1f824-104d-4f37-b265-1c31215c2fe4/3052776d-f0df-4f5c-b23a-46f73ae78b94"
-					(reference "#PWR020")
-					(unit 1)
-				)
-				(path "/32b1f824-104d-4f37-b265-1c31215c2fe4/35fb170e-cc4d-4774-8b9f-87fa9e2bb590"
-					(reference "#PWR025")
+					(reference "#PWR046")
+					(unit 1)
+				)
+				(path "/32b1f824-104d-4f37-b265-1c31215c2fe4/35fb170e-cc4d-4774-8b9f-87fa9e2bb590"
+					(reference "#PWR051")
 					(unit 1)
 				)
@@
 		(on_board yes)
 		(dnp no)
-		(property "Reference" "J3"
+		(property "Reference" "J6"
 			(at 71.374 44.196 0)
 			(effects
@@
 			)
 		)
-		(property "Footprint" ""
+		(property "Footprint" "Connector_USB:USB_C_Receptacle_HCTL_HC-TYPE-C-16P-01A"
 			(at 66.04 63.5 0)
 			(effects
@@
 			(project "RF_HID_module_test"
 				(path "/32b1f824-104d-4f37-b265-1c31215c2fe4/3052776d-f0df-4f5c-b23a-46f73ae78b94"
-					(reference "J3")
-					(unit 1)
-				)
-				(path "/32b1f824-104d-4f37-b265-1c31215c2fe4/35fb170e-cc4d-4774-8b9f-87fa9e2bb590"
-					(reference "J4")
+					(reference "J6")
+					(unit 1)
+				)
+				(path "/32b1f824-104d-4f37-b265-1c31215c2fe4/35fb170e-cc4d-4774-8b9f-87fa9e2bb590"
+					(reference "J7")
 					(unit 1)
 				)
@@
 			)
 		)
-		(property "Footprint" "Marijn_KiCad:ACM2012_TDK_UPDATE"
+		(property "Footprint" "Marijn_KiCad:ACM2012_900_2P_T002_Correct"
 			(at 107.95 71.12 0)
 			(effects
