File: RF_HID_module_test/RF_HID_module_test.kicad_pcb (KiCad board)
At the start: 4 copper layers, 47.5 x 58.8 mm, 67 parts, among them J1 IPX, J2 Conn_02x04_Counter_Clockwise, J3 Conn_ARM_SWD_TagConnect_TC2030, J4 Conn_02x04_Counter_Clockwise, J5 Conn_ARM_SWD_TagConnect_TC2030, J6 CH_USB_C, J7 CH_USB_C, SW1 NRST, SW2 BOOT, SW3 NRST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

Commit message: RF dongle
Routing:
- net GND: track 105.7 -> 117.4 mm, vias 486 -> 488
