File: RF_HID_module_test/RF_HID_module_test.kicad_sch (KiCad schematic)
At the start: 2 parts, among them U2 STM32F412CGUx

Commit message: Schematic V0
Parts:
- added AE1: PCB_ANT, symbol Device:Antenna
- added AE2: 2450AT, symbol Device:Antenna_Chip
- added C1: 2u2, symbol Device:C_Small
- added C10, C11, C14, C15, C16, C17, C8, C9: CL, symbol Device:C_Small
- added C12, C13, C21, C22, C23, C24, C26, C7: 100n, Capacitor_SMD:C_0603_1608Metric, symbol Device:C_Small
- added C18, C25: 4u7, Capacitor_SMD:C_0603_1608Metric, symbol Device:C_Small
- added C19, C20: 1u, Capacitor_SMD:C_0603_1608Metric, symbol Device:C_Small
- added C2: 4u7, symbol Device:C_Small
- added C3, C5: 470n, symbol Device:C_Small
- added C4, C6: 100n, symbol Device:C_Small
- added J1, J2: Conn_ARM_SWD_TagConnect_TC2030, Connector:Tag-Connect_TC2030-IDC-FP_2x03_P1.27mm_Vertical, symbol Connector:Conn_ARM_SWD_TagConnect_TC2030
- added J5: IPX, Connector_Coaxial:U.FL_Molex_MCRF_73412-0110_Vertical, symbol Connector:Conn_Coaxial_Small
- added J6, J7: Conn_02x04_Counter_Clockwise, symbol Connector_Generic:Conn_02x04_Counter_Clockwise
- added L1: 10u, symbol Device:L_Small
- added L2: 10u, Inductor_SMD:L_0805_2012Metric, symbol Device:L_Small
- added R1, R2, R5: 10k, Resistor_SMD:R_0603_1608Metric, symbol Device:R_Small
- added R10, R11, R12: 0, Resistor_SMD:R_0603_1608Metric, symbol Device:R_Small
- added R6, R7, R8, R9: RL, Resistor_SMD:R_0603_1608Metric, symbol Device:R_Small
- added SW1, SW2: NRST, Button_Switch_SMD:SW_SPST_PTS810, symbol Switch:SW_Push
- added SW3: BOOT, Button_Switch_SMD:SW_SPST_PTS810, symbol Switch:SW_Push
- added U5: AP7343, Custom:SOT-25, symbol Marijn:AP7343
- added U6: W25Q128JVS, Marijn_KiCad:SOIC-8_W25QxJVS, symbol Memory_Flash:W25Q128JVS
- added Y1: 32MHz, symbol Device:Crystal_GND24_Small
- added Y2, Y4: 32.786KHz, symbol Device:Crystal_Small
- added Y3: 25MHz, symbol Device:Crystal_GND24_Small
Connections:
- net CH_LSE_I: now reaches U1.1 (A10/LSE32_I)
- net CH_LSE_I: now also C10.2, Y2.1
- net RX: now reaches U1.10 (A9)
- net RX: now also U2.31 (PA10)
- net CH_SWCLK: now reaches U1.11 (B15/TCK)
- net CH_SWCLK: now also J1.4 (SWCLK)
- net CH_SWDIO: now reaches U1.12 (B14/TIO)
- net CH_SWDIO: now also J1.2 (SWDIO)
- net CH_USB/USB_DN: now reaches U1.15 (B11/DP)
- net CH_USB/USB_DP: now reaches U1.16 (B10/DN)
- net CH_O3: now reaches U1.17 (B7)
- net CH_O3: now also J7.4 (Pin_4)
- net CH_O1: now reaches U1.18 (B4)
- net CH_O1: now also J7.2 (Pin_2)
- net CH_NRST: now reaches U1.19 (NRST)
- net CH_NRST: now also C7.2, J1.3 (~{RESET}), R1.1, SW1.1
- net CH_O2: now reaches U1.2 (B6)
- net CH_O2: now also J7.3 (Pin_3)
- net CH_HSE_O: now reaches U1.21 (HSE32_O)
- net CH_HSE_O: now also R8.1
- net CH_HSE_I: now reaches U1.22 (HSE32_I)
- net CH_HSE_I: now also C8.2, Y1.1
- net CH_VINTA: now reaches U1.23 (VINTA)
- net CH_VINTA: now also C5.2, C6.2
- net at U1.24 (ANT): now also R10.2, R11.1, R12.2
- net CH_VDCIA: now reaches U1.25 (VDCIA)
- net CH_VDCIA: now also U1.4 (VDCID), C2.2, C3.2, C4.2, L1.2
- net CH_I0: now reaches U1.26 (A4)
- net CH_I0: now also J7.8 (Pin_8)
- net CH_I1: now reaches U1.27 (A5)
- net CH_I1: now also J7.7 (Pin_7)
- net CH_O0: now reaches U1.3 (B0)
- net CH_O0: now also J7.1 (Pin_1)
- net CH_LSE_O: now reaches U1.32 (A11/LSE32_O)
- net CH_LSE_O: now also R9.1
- net GND: now reaches U1.33 (GND)
- net GND: now also U2.23 (VSS), U2.35 (VSS), U2.47 (VSS), U2.49 (VSS), U2.8 (VSSA), C1.1, C10.1, C11.1, C12.1, C13.1, C14.1, C15.1, C16.1, C17.1, C18.2, C19.2, C2.1, C20.2, C21.2, C22.2, C23.2, C24.2, C25.2, C26.2, C3.1, C4.1, C5.1, C6.1, C7.1, C8.1, C9.1, J1.5 (GND), J2.5 (GND), J5.2 (Ext), R5.1, SW1.2, SW2.2, U5.2 (GND), U6.4 (GND), Y1.2, Y1.4, Y3.2, Y3.4
- net CH_VSW: now reaches U1.5 (VSW)
- net CH_VSW: now also L1.1
- net +3V3: now reaches U1.6 (VDD33)
- net +3V3: now also U2.1 (VBAT), U2.24 (VDD), U2.36 (VDD), U2.48 (VDD), C1.2, C20.1, C21.1, C22.1, C23.1, C24.1, C25.1, J1.1 (VCC), J2.1 (VCC), L2.1, R1.2, R2.2, SW3.1, U5.5 (VOUT), U6.8 (VCC)
- net CH_I2: now reaches U1.7 (A6)
- net CH_I2: now also J7.6 (Pin_6)
- net CH_I3: now reaches U1.8 (A7)
- net CH_I3: now also J7.5 (Pin_5)
- net TX: now reaches U1.9 (A8)
- net TX: now also U2.38 (PA15)
- net FLASH_SPI_NCS: now reaches U2.14 (PA4)
- net FLASH_SPI_NCS: now also U6.1 (~{CS})
- net FLASH_SPI_CLK: now reaches U2.15 (PA5)
- net FLASH_SPI_CLK: now also U6.6 (CLK)
- net FLASH_SPI_MISO: now reaches U2.16 (PA6)
- net FLASH_SPI_MISO: now also U6.2 (DO(IO1))
- net FLASH_SPI_MOSI: now reaches U2.17 (PA7)
- net FLASH_SPI_MOSI: now also U6.5 (DI(IO0))
- net STM_O0: now reaches U2.18 (PB0)
- net STM_O0: now also J6.1 (Pin_1)
- net STM_O1: now reaches U2.19 (PB1)
- net STM_O1: now also J6.2 (Pin_2)
- net STM_O2: now reaches U2.20 (PB2)
- net STM_O2: now also J6.3 (Pin_3)
- net at U2.22 (VCAP_1): now also C18.1
- net W25Q128_NRST: now reaches U2.29 (PA8)
- net W25Q128_NRST: now also U6.7 (IO3)
- net STM_LSE_I: now reaches U2.3 (PC14)
- net STM_LSE_I: now also C16.2, Y4.1
- net W25Q128_NWP: now reaches U2.30 (PA9)
- net W25Q128_NWP: now also U6.3 (IO2)
- net STM_USB/USB_DN: now reaches U2.32 (PA11)
- net STM_USB/USB_DP: now reaches U2.33 (PA12)
- net STM_SWDIO: now reaches U2.34 (PA13)
- net STM_SWDIO: now also J2.2 (SWDIO)
- net STM_SWCLK: now reaches U2.37 (PA14)
- net STM_SWCLK: now also J2.4 (SWCLK)
- net STM_O3: now reaches U2.39 (PB3)
- net STM_O3: now also J6.4 (Pin_4)
- net STM_LSE_O: now reaches U2.4 (PC15)
- net STM_LSE_O: now also R7.1
- net STM_I0: now reaches U2.40 (PB4)
- net STM_I0: now also J6.8 (Pin_8)
- net STM_I1: now reaches U2.41 (PB5)
- net STM_I1: now also J6.7 (Pin_7)
- net STM_I2: now reaches U2.42 (PB6)
- net STM_I2: now also J6.6 (Pin_6)
- net STM_I3: now reaches U2.43 (PB7)
- net STM_I3: now also J6.5 (Pin_5)
- net STM_BOOT: now reaches U2.44 (BOOT0)
- net STM_BOOT: now also C13.2, R5.2, SW3.2
- net STM_HSE_I: now reaches U2.5 (PH0)
- net STM_HSE_I: now also C14.2, Y3.1
- net STM_HSE_O: now reaches U2.6 (PH1)
- net STM_HSE_O: now also R6.1
- net STM_NRST: now reaches U2.7 (NRST)
- net STM_NRST: now also C12.2, J2.3 (~{RESET}), R2.1, SW2.1
- net +3.3VA: now reaches U2.9 (VDDA)
- net +3.3VA: now also C26.1, L2.2
- new net: AE1.1 (A), R10.1
- new net: C15.2, R6.2, Y3.3
- new net: C11.2, R9.2, Y2.2
- new net: C9.2, R8.2, Y1.3
- new net: J5.1 (In), R12.1
- new net: AE2.1 (FEED), R11.2
- new net: C17.2, R7.2, Y4.2
- new net +5V: C19.1, U5.1 (VIN), U5.3 (EN)
- no-connect marks 0 -> 21
Other:
- added sheet CH_USB (USB.kicad_sch)
- added sheet STM_USB (USB.kicad_sch)
- note added: "3v3 LDO"
- note added: "Bypass for CH"
- note added: "Bypass/filter for STM"
- note added: "JTAG, NRST and OSC for CH"
- note added: "JTAG, NRST/BOOT and OSC for STM"
- note added: "Key grid connectors"
- note added: "SPI flash (W25Q128)"
- moved on the sheet: U2

Commit message: Layout V0
Parts:
- removed AE2: 2450AT, symbol Device:Antenna_Chip
- removed C10, C8, C9: CL, symbol Device:C_Small
- removed C13, C22: 100n, Capacitor_SMD:C_0603_1608Metric, symbol Device:C_Small
- removed C19, C20: 1u, Capacitor_SMD:C_0603_1608Metric, symbol Device:C_Small
- removed C5: 470n, symbol Device:C_Small
- removed C6: 100n, symbol Device:C_Small
- removed R8: RL, Resistor_SMD:R_0603_1608Metric, symbol Device:R_Small
- removed U5: AP7343, Custom:SOT-25, symbol Marijn:AP7343
- added AE2: 2450AT18D0100, Marijn_KiCad:2450AT18D0100, symbol Marijn:2450AT18D0100
- added C12: 100n, Capacitor_SMD:C_0603_1608Metric, symbol Device:C_Small
- added C14: 10u, Capacitor_SMD:C_0603_1608Metric, symbol Device:C_Small
- added C15: 56p, Capacitor_SMD:C_0603_1608Metric, symbol Device:C_Small
- added C16, C17: 22u, Capacitor_SMD:C_0603_1608Metric, symbol Device:C_Small
- added D1: PWR, LED_SMD:LED_0603_1608Metric, symbol Device:LED
- added D2: CH_STATUS, LED_SMD:LED_0603_1608Metric, symbol Device:LED
- added D3: STM_STATUS, LED_SMD:LED_0603_1608Metric, symbol Device:LED
- added L3: 1u, Inductor_SMD:L_APV_ANR4018, symbol Device:L_Small
- added R11: 320k, Resistor_SMD:R_0603_1608Metric, symbol Device:R_Small
- added R5: 5k1, Resistor_SMD:R_0603_1608Metric, symbol Device:R_Small
- added TP1: 3V3, TestPoint:TestPoint_Pad_D1.5mm, symbol Connector:TestPoint
- added U3: ISL91127IRAZ, Package_DFN_QFN:QFN-20-1EP_4x4mm_P0.5mm_EP2.7x2.7mm_ThermalVias, symbol Marijn:ISL91127IR
- added U5: W25Q128JVS, Marijn_KiCad:SOIC-8_W25QxJVS, symbol Memory_Flash:W25Q128JVS
- AE1: footprint (none) -> RF_Antenna:Texas_SWRA117D_2.4GHz_Left
- C10: renamed from C4; footprint (none) -> Capacitor_SMD:C_0603_1608Metric
- C11: value CL -> 470n; footprint (none) -> Capacitor_SMD:C_0603_1608Metric
- C19: renamed from C14; value CL -> 12p; footprint (none) -> Capacitor_SMD:C_0603_1608Metric
- C20: renamed from C15; value CL -> 12p; footprint (none) -> Capacitor_SMD:C_0603_1608Metric
- C21: renamed from C16; value CL -> 12p; footprint (none) -> Capacitor_SMD:C_0603_1608Metric
- C22: renamed from C17; value CL -> 12p; footprint (none) -> Capacitor_SMD:C_0603_1608Metric
- C7: renamed from C1; footprint (none) -> Capacitor_SMD:C_0603_1608Metric
- C8: renamed from C2; footprint (none) -> Capacitor_SMD:C_0603_1608Metric
- C9: renamed from C3; footprint (none) -> Capacitor_SMD:C_0603_1608Metric
- J2: renamed from J7; footprint (none) -> Connector_PinSocket_2.54mm:PinSocket_2x04_P2.54mm_Vertical
- J4: renamed from J6; footprint (none) -> Connector_PinSocket_2.54mm:PinSocket_2x04_P2.54mm_Vertical
- L2: renamed from L1; footprint (none) -> Inductor_SMD:L_0805_2012Metric
- R6, R7: value RL -> 1k; LCSC C25118 -> (none); mouser (none) -> 71-CRCW06031K00FKEE
- R9: value RL -> 1M; LCSC C25118 -> (none); mouser (none) -> 791-RMC1/16-512JTP
- Y1: renamed from Y2; footprint (none) -> Crystal:Crystal_SMD_3215-2Pin_3.2x1.5mm
- Y2: renamed from Y1; footprint (none) -> Crystal:Crystal_SMD_3225-4Pin_3.2x2.5mm
- Y3: footprint (none) -> Crystal:Crystal_SMD_3225-4Pin_3.2x2.5mm
- Y4: footprint (none) -> Crystal:Crystal_SMD_3215-2Pin_3.2x1.5mm
- renumbered C18 to C1, C7 to C13, C12 to C18, C21 to C2, C23 to C3, C24 to C4, C25 to C5, C26 to C6, J5 to J1, J1 to J3, J2 to J5, L2 to L1, R10 to R1, R5 to R10, R11 to R2, R12 to R3, R1 to R4, R2 to R8, SW3 to SW2, SW2 to SW3, U6 to U4
Connections:
- net +3V3: now also R6.1, R7.1, R9.1, C15.1, C16.1, C17.1, R5.1, TP1.1, U3.17 (VOUT), U3.18 (VOUT), U3.19 (VOUT), U3.20 (VOUT), U5.8 (VCC)
- net +5V: now also C14.1, U3.10 (VIN), U3.11 (EN), U3.12 (MODE), U3.6 (PVIN), U3.7 (PVIN), U3.8 (PVIN), U3.9 (PVIN)
- net CH_HSE_O: now also Y2.3
- net CH_LSE_O: now also Y1.2; no longer R9.1
- net CH_USB/USB_DN: now also U1.16 (B10/DN); no longer U1.15 (B11/DP)
- net CH_USB/USB_DP: now also U1.15 (B11/DP); no longer U1.16 (B10/DN)
- net CH_VINTA: now also C11.2, C12.2
- net GND: now also AE2.2, AE2.3, AE2.4, C12.1, C14.2, C16.2, C17.2, D1.1 (K), R11.1, U3.13 (SGND), U3.14 (SGND), U3.21 (EPAD), U3.3 (PGND), U5.4 (GND)
- net STM_HSE_O: now also C20.2, Y3.3; no longer R6.1
- net STM_LSE_O: now also C22.2, Y4.2; no longer R7.1
- net STM_SWO: now reaches J5.6 (SWO)
- net STM_SWO: now also U2.39 (PB3)
- net CH_W25Q128_NRST: now reaches U1.13 (B13)
- net CH_W25Q128_NRST: now also U5.7 (IO3)
- net CH_W25Q128_NWP: now reaches U1.14 (B12)
- net CH_W25Q128_NWP: now also U5.3 (IO2)
- net CH_STATUS: now reaches U1.20 (B22)
- net CH_STATUS: now also D2.1 (K)
- net CH_FLASH_SPI_MISO: now reaches U1.28 (A15)
- net CH_FLASH_SPI_MISO: now also U5.2 (DO(IO1))
- net CH_FLASH_SPI_MOSI: now reaches U1.29 (A14)
- net CH_FLASH_SPI_MOSI: now also U5.5 (DI(IO0))
- net CH_FLASH_SPI_CLK: now reaches U1.30 (A13)
- net CH_FLASH_SPI_CLK: now also U5.6 (CLK)
- net CH_FLASH_SPI_NCS: now reaches U1.31 (A12)
- net CH_FLASH_SPI_NCS: now also U5.1 (~{CS})
- net at R2.2: now also AE2.1 (FEED)
- net STM_IO0: now reaches U2.10 (PA0)
- net STM_IO0: now also J4.1 (Pin_1)
- net STM_IO1: now reaches U2.11 (PA1)
- net STM_IO1: now also J4.2 (Pin_2)
- net STM_IO2: now reaches U2.12 (PA2)
- net STM_IO2: now also J4.3 (Pin_3)
- net STM_IO3: now reaches U2.13 (PA3)
- net STM_IO3: now also J4.4 (Pin_4)
- net CH_I0 renamed CH_IO4
- net CH_IO4: now also J2.5 (Pin_5); no longer J2.8 (Pin_8)
- net CH_I1 renamed CH_IO5
- net CH_IO5: now also J2.6 (Pin_6); no longer J2.7 (Pin_7)
- net CH_I2 renamed CH_IO6
- net CH_IO6: now also J2.7 (Pin_7); no longer J2.6 (Pin_6)
- net CH_I3 renamed CH_IO7
- net CH_IO7: now also J2.8 (Pin_8); no longer J2.5 (Pin_5)
- net CH_O0 renamed CH_IO0
- net CH_O1 renamed CH_IO1
- net CH_O2 renamed CH_IO2
- net CH_O3 renamed CH_IO3
- net FLASH_SPI_CLK renamed STM_FLASH_SPI_CLK
- net FLASH_SPI_MISO renamed STM_FLASH_SPI_MISO
- net FLASH_SPI_MOSI renamed STM_FLASH_SPI_MOSI
- net FLASH_SPI_NCS renamed STM_FLASH_SPI_NCS
- net STM_I0 renamed STM_IO4
- net STM_IO4: now also J4.5 (Pin_5); no longer J4.8 (Pin_8)
- net STM_I1 renamed STM_IO5
- net STM_IO5: now also J4.6 (Pin_6); no longer J4.7 (Pin_7)
- net STM_I2 renamed STM_IO6
- net STM_IO6: now also J4.7 (Pin_7); no longer J4.6 (Pin_6)
- net STM_I3 renamed STM_IO7
- net STM_IO7: now also J4.8 (Pin_8); no longer J4.5 (Pin_5)
- net STM_O0 renamed STM_STATUS
- net STM_STATUS: now also D3.1 (K); no longer J4.1 (Pin_1)
- net STM_O1: no longer names the net of U2.19 (PB1)
- net STM_O1: no longer J4.2 (Pin_2)
- net STM_O2: no longer names the net of U2.20 (PB2)
- net STM_O2: no longer J4.3 (Pin_3)
- removed net STM_O3: J4.4 (Pin_4), U2.39 (PB3)
- net W25Q128_NRST renamed STM_W25Q128_NRST
- net W25Q128_NWP renamed STM_W25Q128_NWP
- new net: C15.2, R11.2, R9.2, U3.15 (FB)
- new net: L3.2, U3.1 (LX2), U3.2 (LX2)
- new net: L3.1, U3.4 (LX1), U3.5 (LX1)
- new net: D3.2 (A), R7.2
- new net: D2.2 (A), R6.2
- new net: D1.2 (A), R5.2
- no-connect marks 21 -> 10
Other:
- note added: "GPIO"
- note added: "LEDs"
- note added: "PWR"
- note added: "https://orbcode.org/orbuculum/single-wire-output/"
- note added: "include a GND guard band around the feedback resistor network"
- note removed: "3v3 LDO"
- note removed: "Key grid connectors"
- moved on the sheet: C2, C3, C4, C5, C6, J2, J4, L1, R10, SW2, Y1, Y2

Commit message: RF dongle
Connections:
- no-connect marks 10 -> 11
Changed lines of the file:
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@@
 		(at 45.72 110.49)
+	)
+	(no_connect
+		(at 45.72 72.39)
 	)
 	(wire
