File: RF_HID_dongle_test/RF_HID_dongle_test.kicad_sch (KiCad schematic)
At the start: 25 parts, among them J1 PCB_USB, J2 Conn_ARM_SWD_TagConnect_TC2030, U3 AP7343, Y2 32MHz

Commit message: EOL for WCH chips
Changed lines of the file:
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@@
 (kicad_sch
-	(version 20231120)
+	(version 20250114)
 	(generator "eeschema")
-	(generator_version "8.0")
+	(generator_version "9.0")
 	(paper "A4")
 	(junction
@@
 		)
 	)
+	(embedded_fonts no)
 )
